File: root_hub.kicad_sch (KiCad schematic)
At the start: 19 parts, among them U201 USB2514B, Y201 24Mhz

Commit message: Add power management
And also some random stuff here and there
Parts:
- removed C207: 4.7uF, Capacitor_SMD:C_0603_1608Metric, symbol Device:C
- removed C209, C210: 100nF, Capacitor_SMD:C_0402_1005Metric, symbol Device:C
- removed U201: USB2514B, Package_DFN_QFN:QFN-36-1EP_6x6mm_P0.5mm_EP3.7x3.7mm, symbol Interface_USB:USB2514B_Bi
- added C213, C215, C217: 100nF, Capacitor_SMD:C_0402_1005Metric, symbol Device:C
- added C214, C216: 1.0uF, Capacitor_SMD:C_0603_1608Metric, symbol Device:C
- added C218, C219: 1.0uF, Capacitor_SMD:C_0402_1005Metric, symbol Device:C
- added IC201: USB2517, Package_DFN_QFN:QFN-64-1EP_9x9mm_P0.5mm_EP4.7x4.7mm_ThermalVias, symbol fabian_usb:USB2517
- added J201: Barrel_Jack, Capacitor_SMD:C_0603_1608Metric, symbol Connector:Barrel_Jack
- added P201: USB_C_Plug_USB2.0, Connector_USB:USB_C_Receptacle_G-Switch_GT-USB-7010ASV, symbol Connector:USB_C_Plug_USB2.0
- added R206, R207: 5.1k, Resistor_SMD:R_0402_1005Metric, symbol Device:R
- added U201: SRV05-4, Package_TO_SOT_SMD:SOT-23-6, symbol Power_Protection:SRV05-4
Connections:
- net +3V3: now also C217.1, C218.1, C219.1, IC201.10 (VDDA33), IC201.24 (VDD33CR), IC201.46 (VDD33), IC201.5 (VDDA33), IC201.52 (VDDA33), IC201.57 (VDDA33), IC201.64 (VDD33PLL)
- net D+: now also IC201.59 (USBUP_DP)
- net D-: now also IC201.58 (USBUP_DM)
- net GND: now also C213.2, C214.2, C215.2, C216.2, C217.2, C218.2, C219.2, IC201.19 (TEST), IC201.65 (EP), J201.2, P201.A1 (GND), P201.A12 (GND), P201.B1 (GND), P201.B12 (GND), R206.2, R207.2, U201.2 (VN)
- net VBUS: now also P201.A4 (VBUS), P201.A9 (VBUS), P201.B4 (VBUS), P201.B9 (VBUS), U201.5 (VP)
- net VBUS_DET: now also IC201.44 (VBUS_DET)
- net XTAL_IN: now also IC201.61 (XTAL1/CLKIN)
- net XTAL_OUT: now also IC201.60 (XTAL2)
- net at R204.2: now also IC201.63 (RBIAS)
- net RESET_N: now reaches C208.1, R202.2
- net RESET_N: now also IC201.43 (RESET_N)
- new net: P201.A5 (CC), R207.1
- new net: C213.1, C214.1, IC201.62 (VDD18PLL)
- new net: C215.1, C216.1, IC201.25 (VDD18)
- new net: P201.A6 (D+), U201.1 (IO1)
- new net: P201.A7 (D-), U201.3 (IO2)
- new net: P201.B5 (VCONN), R206.1
- new net +5V: J201.1
- new net Earth: P201.S1 (SHIELD)
- new net Port 1-2/PORT_A_EN_1: IC201.29 (PRTPWR1)
- new net Port 1-2/PORT_A_OC: IC201.28 (OCS1_N)
- new net Port 1-2/PORT_B_EN_1: IC201.26 (PRTPWR2)
- new net Port 1-2/PORT_B_OC: IC201.27 (OCS2_N)
- new net Port 1-2/USB_A_D+: IC201.2 (USBDN1_DP/PRT_DIS_P1)
- new net Port 1-2/USB_A_D-: IC201.1 (USBDN1_DM/PRT_DIS_M1)
- new net Port 1-2/USB_B_D+: IC201.4 (USBDN2_DP/PRT_DIS_P2)
- new net Port 1-2/USB_B_D-: IC201.3 (USBDN2_DM/PRT_DIS_M2)
- new net Port 3-4/PORT_A_EN_1: IC201.23 (PRTPWR3)
- new net Port 3-4/PORT_A_OC: IC201.22 (OCS3_N)
- new net Port 3-4/PORT_B_EN_1: IC201.20 (PRTPWR4)
- new net Port 3-4/PORT_B_OC: IC201.21 (OCS4_N)
- new net Port 3-4/USB_A_D+: IC201.7 (USBDN3_DP/PRT_DIS_P3)
- new net Port 3-4/USB_A_D-: IC201.6 (USBDN3_DM/PRT_DIS_M3)
- new net Port 3-4/USB_B_D+: IC201.9 (USBDN4_DP/PRT_DIS_P4)
- new net Port 3-4/USB_B_D-: IC201.8 (USBDN4_DM/PRT_DIS_M4)
- new net Port 5-6/PORT_A_EN_1: IC201.30 (PRTPWR5)
- new net Port 5-6/PORT_A_OC: IC201.35 (OCS5_N)
- new net Port 5-6/PORT_B_EN_1: IC201.39 (PRTPWR6)
- new net Port 5-6/PORT_B_OC: IC201.38 (OCS6_N)
- new net Port 5-6/USB_A_D+: IC201.12 (USBDN5_DP/PRT_DIS_P5)
- new net Port 5-6/USB_A_D-: IC201.11 (USBDN5_DM/PRT_DIS_M5)
- new net Port 5-6/USB_B_D+: IC201.54 (USBDN6_DP/PRT_DIS_P6)
- new net Port 5-6/USB_B_D-: IC201.53 (USBDN6_DM/PRT_DIS_M6)
- new net Power controller/USB_DM: IC201.55 (USBDN7_DM/PRT_DIS_M7)
- new net Power controller/USB_DP: IC201.56 (USBDN7_DP/PRT_DIS_P7)
- no-connect marks 0 -> 2
Other:
- added sheet Port 1-2 (dual_outports.kicad_sch)
- added sheet Port 3-4 (dual_outports.kicad_sch)
- added sheet Port 5-6 (dual_outports.kicad_sch)
- added sheet Power (power.kicad_sch)
- added sheet Power controller (controller.kicad_sch)
- moved on the sheet: C208, C211, C212, R201, R202, R203, R204, R205, Y201
