File: usb-hub.kicad_sch (KiCad schematic)
At the start: 37 parts, among them IC101 USB2517, J101 Barrel_Jack_Switch, J102 USB_C_Receptacle_USB2.0_14P, U101 USBLC6-2P6, Y101 24Mhz

Commit message: Commit old worktree
Parts:
- R101: value 420k -> 100k
Changed lines of the file:
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@@
 		(fields_autoplaced yes)
 		(property "Reference" "R101"
-			(at 179.07 44.4499 0)
+			(at 179.07 44.45 0)
 			(effects
 				(font
@@
 			)
 		)
-		(property "Value" "420k"
-			(at 179.07 46.9899 0)
+		(property "Value" "100k"
+			(at 179.07 46.99 0)
 			(effects
 				(font
